File: cad/timer.kicad_pcb (KiCad board)
At the start: 2 copper layers, 47 x 47 mm, 22 parts, among them J1 Motor, J2 Pot, J4 Prog, Q1 S9012, Q2 S9013, Q3 S9012, U1 ATMEGA328P-PU, U2 LM393, U3 L293D, Y1 32.768kHz

Commit message: CAD changes for off stop size change
The soft power switch needs a 68k instead of a 47k resistor now.
Parts:
- R2: value 47kΩ -> 68kΩ
Changed lines of the file:
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@@
       (effects (font (size 1 1) (thickness 0.15)))
     )
-    (fp_text value 47kΩ (at 5.08 -2.54 450) (layer F.Fab)
+    (fp_text value 68kΩ (at 5.08 -2.54 450) (layer F.Fab)
       (effects (font (size 1 1) (thickness 0.15)))
     )
