File: cad/timer.kicad_sch (KiCad schematic)
At the start: 25 parts, among them U2 LM393

Commit message: Update CAD for redesign
Also cleanup old files in cad directory
Parts:
- removed C2: (no value), symbol Device:C
- removed R2: (no value), symbol Device:R
- removed U2: LM393, Housings_DIP:DIP-8_W7.62mm, symbol timer-rescue:LM393
- added C3: 100nF, Capacitor_THT:C_Disc_D5.0mm_W2.5mm_P5.00mm, symbol Device:C
- added D1: 1N5819, Diode_THT:D_DO-41_SOD81_P2.54mm_Vertical_KathodeUp, symbol Device:D
- added R3: 4.7Ω, Resistor_THT:R_Axial_DIN0207_L6.3mm_D2.5mm_P2.54mm_Vertical, symbol Device:R
- added R4: 100kΩ, Resistor_THT:R_Axial_DIN0207_L6.3mm_D2.5mm_P2.54mm_Vertical, symbol Device:R
- BT1: value (none) -> Battery; footprint (none) -> Connector_PinHeader_2.54mm:PinHeader_1x02_P2.54mm_Vertical
- C1: value 10uF -> 470µF; footprint Capacitors_THT:CP_Radial_D5.0mm_P2.50mm -> Capacitor_THT:CP_Radial_D10.0mm_P5.00mm
- C2: renamed from C5; value (none) -> 100nF; footprint (none) -> Capacitor_THT:C_Disc_D5.0mm_W2.5mm_P5.00mm
- C4: renamed from C3; value (none) -> 100nF; footprint (none) -> Capacitor_THT:C_Disc_D5.0mm_W2.5mm_P5.00mm
- C5: renamed from C6; value (none) -> 100nF; footprint (none) -> Capacitor_THT:C_Disc_D5.0mm_W2.5mm_P5.00mm
- C6: renamed from C4; value (none) -> 100nF; footprint (none) -> Capacitor_THT:C_Disc_D5.0mm_W2.5mm_P5.00mm
- C7: renamed from C9; value (none) -> 15pF; footprint (none) -> Capacitor_THT:C_Disc_D5.0mm_W2.5mm_P2.50mm
- C8: value (none) -> 15pF; footprint (none) -> Capacitor_THT:C_Disc_D5.0mm_W2.5mm_P2.50mm
- C9: renamed from C7; value (none) -> 47pF; footprint (none) -> Capacitor_THT:C_Disc_D5.0mm_W2.5mm_P2.50mm
- D2: renamed from D1; value (none) -> 1N5819; footprint (none) -> Diode_THT:D_DO-41_SOD81_P2.54mm_Vertical_KathodeUp
- D3: renamed from D2; value (none) -> 1N5819; footprint (none) -> Diode_THT:D_DO-41_SOD81_P2.54mm_Vertical_KathodeUp
- MT1: value (none) -> Motor; footprint (none) -> Connector_PinHeader_2.54mm:PinHeader_1x02_P2.54mm_Vertical
- PR1: value (none) -> Prog; footprint (none) -> Connector_PinHeader_2.54mm:PinHeader_1x03_P2.54mm_Vertical
- Q1, Q2: value (none) -> BS170; footprint (none) -> Package_TO_SOT_THT:TO-92_Inline_Wide
- R1: value (none) -> 100kΩ; footprint (none) -> Resistor_THT:R_Axial_DIN0207_L6.3mm_D2.5mm_P2.54mm_Vertical
- R2: renamed from R3; value (none) -> 1kΩ; footprint (none) -> Resistor_THT:R_Axial_DIN0207_L6.3mm_D2.5mm_P2.54mm_Vertical
- R5: renamed from R4; value (none) -> 1kΩ; footprint (none) -> Resistor_THT:R_Axial_DIN0207_L6.3mm_D2.5mm_P2.54mm_Vertical
- SP1: value (none) -> Speaker; footprint (none) -> Connector_PinHeader_2.54mm:PinHeader_1x02_P2.54mm_Vertical
- U1: value (none) -> ATMEGA328P-PU; footprint (none) -> Package_DIP:DIP-28_W7.62mm_Socket
- VR1: value (none) -> Pot; footprint (none) -> Connector_PinHeader_2.54mm:PinHeader_1x03_P2.54mm_Vertical
- Y1: value (none) -> 32.768kHz; footprint (none) -> Crystal:Crystal_C38-LF_D3.0mm_L8.0mm_Vertical
Connections:
- net GND: now also R1.2, R4.2; no longer VR1.3 (Pin_3)
- net VCC: now also MT1.1 (Pin_1), C3.1, D1.1 (K), R3.1; no longer BT1.1 (+), C5.1, D3.1 (K), MT1.2 (Pin_2), R1.2, SP1.1
- net at U1.4 ((PCINT18/INT0)PD2): now also R2.2
- net at R1.1: now also Q1.2 (G), R2.1
- net at U1.18 ((PCINT4/MISO)PB4): no longer R2.2
- net at U1.24 ((PCINT9/ADC1)PC1): now also VR1.3 (Pin_3), C3.2
- net at D2.2 (A), Q1.1 (D): now also MT1.2 (Pin_2); no longer MT1.1 (Pin_1)
- net at Q2.2 (G), R5.1: now also R4.1
- new net: C5.1, D3.1 (K), R3.2, SP1.1
- new net: BT1.1 (+), D1.2 (A)
Other:
- note removed: "Soft Power Switch"
- moved on the sheet: BT1, C1, R2, R5, VR1
